File: Projects/StepUp/StepUp.kicad_sch (KiCad schematic)
At the start: 9 parts

Commit message: feat(v0.4): Work in Progress
Other:
- note added: "M3 for threaded inserts + bolts M2 for board support (no bolts)"
- note removed: "M3 for threaded inserts M2 for board support"
Changed lines of the file:
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@@
 		(title "System diagram")
 		(date "2025-03-03")
-		(rev "v0.3")
+		(rev "v0.4")
 		(company "SJFOM")
 	)
@@
 		)
 	)
-	(text "M3 for threaded inserts\nM2 for board support"
+	(text "M3 for threaded inserts + bolts\nM2 for board support (no bolts)"
 		(exclude_from_sim no)
 		(at 26.416 154.432 0)
@@
 				)
 				(justify left)
+				(hide yes)
 			)
 		)
@@
 				)
 				(justify left)
+				(hide yes)
 			)
 		)
@@
 				)
 				(justify left)
+				(hide yes)
 			)
 		)
@@
 				)
 				(justify left)
+				(hide yes)
 			)
 		)
@@
 				)
 				(justify left)
+				(hide yes)
 			)
 		)
@@
 				)
 				(justify left)
+				(hide yes)
 			)
 		)
@@
 				)
 				(justify left)
+				(hide yes)
 			)
 		)
@@
 				)
 				(justify left)
+				(hide yes)
 			)
 		)
@@
 				)
 				(justify left)
-			)
-		)
+				(hide yes)
+			)
+		)
