File: Projects/StepUp/indicators.kicad_sch (KiCad schematic)
At the start: 10 parts, among them Q7 2N7002-7-F

Commit message: feat(v1.0): Migrate v0.4 to v1.0
Parts:
- removed R54: 100kR, Resistor_SMD:R_0603_1608Metric, symbol Device:R
- added R52: 100kR, Resistor_SMD:R_0603_1608Metric, symbol Device:R
- BZ1: PLACE_BY_HAND (none) -> Y
- renumbered Q7 to Q6, R49 to R47, R50 to R48, R51 to R49, R52 to R50, R53 to R51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
Connections:
- net GND: now also R52.2
- net at Q6.1 (G), R51.2: now also R52.1
